File: MegaCD-837-8015-Rev0-MCE1/MegaCD.kicad_pcb (KiCad board)
At the start: 4 copper layers, 188.9 x 92 mm, 107 parts, among them CN1 CON 25P ANGLE, CN2 EDGE 60P, CN3 CON 21P, IC1 68HC000, IC10 MB8464A-10L, IC11 TC511664BZ, IC12 TC511664BZ, IC13 65256BLFP-10T, IC14 65256BLFP-10T, IC15 LC8951, IC16 74HC00, IC17 MB8464A-90L, IC18 MB8464A-90L, IC19 74HC112, IC2 315-5477, IC20 74HC245, IC3 315-5476, IC4 27C1024, IC5 MB81C4256Z, IC6 MB81C4256Z, IC7 MB81C4256Z, IC8 MB81C4256Z, IC9 MB3790, M0 TestPoint, M1 TestPoint, M10 TestPoint, M11 TestPoint, M2 TestPoint, M3 TestPoint, M4 TestPoint, M5 TestPoint, M6 TestPoint, M7 TestPoint, M8 TestPoint, M9 TestPoint

Commit message: Improve board design by making it possible to mostly manufacture at JLCPCB
Parts:
- C10, C11, C12, C13, C23, C28, C31, C37, C41, C42, C46, C9: footprint MegaCD_Footprints:CP_Elec_3x5.4 -> MegaCD_Footprints:CP_Elec_4x5.4
- IC16: footprint MegaCD_Footprints:SOIC-14W_5.3mm_P1.27mm -> MegaCD_Footprints:IC_SN74HC00DR
- IC19: footprint MegaCD_Footprints:SOIC-16W_5.3x10.2mm_P1.27mm -> MegaCD_Footprints:IC_SN74HC112DR
- moved C9 0.76 mm to (118.1, 84.9)
- moved C12 0.76 mm to (149.9, 117.5)
- moved C41 0.52 mm to (59.6, 83.7)
- moved C11 0.51 mm to (177.9, 126.1)
- moved C13 0.51 mm to (149.9, 107.6)
- moved C42 0.44 mm to (65.4, 57.9)
- moved C10 0.13 mm to (149.9, 112.5)
- moved FB5 0.09 mm to (163.1, 118.6)
Connections:
- net Net-(BT1-+) renamed /VBAT
- net Net-(CN1-Pin_10) renamed /C2PO
- net Net-(CN1-Pin_17) renamed /EXCK
- net Net-(CN1-Pin_2) renamed /D/M
- net Net-(CN1-Pin_3) renamed /~{IRQ}
- net Net-(CN1-Pin_5) renamed /HDCK
- net Net-(CN1-Pin_6) renamed /DB0
- net Net-(CN1-Pin_7) renamed /DB1
- net Net-(CN1-Pin_8) renamed /DB2
- net Net-(CN1-Pin_9) renamed /DB3
- net Net-(CN3-Pin_19) renamed /VCC2F
- net Net-(IC10-CS2) renamed /~{NVRAM_RESET}
- net Net-(IC10-VCC) renamed /NVRAM_VCC
- net Net-(IC11-A0) renamed /EAD0
- net Net-(IC11-A1) renamed /EAD1
- net Net-(IC11-A2) renamed /EAD2
- net Net-(IC11-A3) renamed /EAD3
- net Net-(IC11-A4) renamed /EAD4
- net Net-(IC11-A5) renamed /EAD5
- net Net-(IC11-A6) renamed /EAD6
- net Net-(IC11-A7) renamed /EAD7
- net Net-(IC11-D10) renamed /ED10
- net Net-(IC11-D11) renamed /ED11
- net Net-(IC11-D12) renamed /ED12
- net Net-(IC11-D13) renamed /ED13
- net Net-(IC11-D14) renamed /ED14
- net Net-(IC11-D15) renamed /ED15
- net Net-(IC11-D8) renamed /ED8
- net Net-(IC11-D9) renamed /ED9
- net Net-(IC12-A0) renamed /OAD0
- net Net-(IC12-A1) renamed /OAD1
- net Net-(IC12-A2) renamed /OAD2
- net Net-(IC12-A3) renamed /OAD3
- net Net-(IC12-A4) renamed /OAD4
- net Net-(IC12-A5) renamed /OAD5
- net Net-(IC12-A6) renamed /OAD6
- net Net-(IC12-A7) renamed /OAD7
- net Net-(IC12-D10) renamed /OD10
- net Net-(IC12-D11) renamed /OD11
- net Net-(IC12-D12) renamed /OD12
- net Net-(IC12-D13) renamed /OD13
- net Net-(IC12-D14) renamed /OD14
- net Net-(IC12-D15) renamed /OD15
- net Net-(IC12-D8) renamed /OD8
- net Net-(IC12-D9) renamed /OD9
- net Net-(IC13-~{WE}) renamed /~{RWE}
- net Net-(IC15-~{RCS}) renamed /~{RCS}
- net Net-(IC15-~{ROE}) renamed /~{ROE8951}
- net Net-(IC15-~{RWE}) renamed /~{RWE8951}
- net Net-(IC19A-Q) renamed /~{RCS1Q}
- net Net-(IC19A-~{R}) renamed /~{RCS1N}
- net Net-(IC19B-Q) renamed /~{RCS2Q}
- net Net-(IC19B-~{R}) renamed /~{RCS2N}
- net Net-(IC2-12M) renamed /12MF
- net Net-(IC2-25M) renamed /25MF
- net Net-(IC2-LEDG) renamed /LEDG
- net Net-(IC2-LEDR) renamed /LEDR
- net Net-(IC9-CT) renamed /BATPW
- net Net-(LD1-A) renamed /LD1A
- net Net-(LD1-K) renamed /LD1K
- net Net-(LD2-A) renamed /LD2A
- net Net-(LD2-K) renamed /LD2K
- net Net-(OSC1-OUT) renamed /50MF
- net Net-(TR1-B) renamed /LD2TRB
- net Net-(TR2-B) renamed /LD1TRB
Routing:
- net GND: track 2387.6 -> 2409.4 mm
- net VCC2: track 1456.3 -> 1466.2 mm
- net SR2: track 96.8 -> 101.0 mm
- net ~{ROE}: track 65.6 -> 68.0 mm
- net ~{RCS2X}: track 34.1 -> 32.1 mm
- net BCK: track 76.6 -> 74.7 mm
- net /~{RCS1Q}: track 43.9 -> 42.2 mm
- net /~{RCS2N}: track 47.5 -> 48.9 mm
- net BCLKB: track 225.4 -> 226.7 mm
- net ~{RCS1X}: track 29.4 -> 28.0 mm
- net /~{RCS1N}: track 46.6 -> 45.5 mm
- net 25M: track 52.6 -> 51.6 mm
- net /~{RCS2Q}: track 39.6 -> 40.4 mm
- net ~{ECAS}: track 68.7 -> 68.0 mm
- net ~{RCS2}: track 53.8 -> 53.1 mm
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- added copper zone on In4.Cu, net GND
- added copper zone on In3.Cu, net VCC2
Other:
- copper layers 4 -> 6
- board text added: "BY COSAM B VER BY ZIGGY"
- board text added: "E"
- board text added: "FC0"
- board text added: "FC1"
- board text added: "REPRO v1.2B BY COSAM / B VER BY ZIGGY"
- board text added: "TRANS RIGHTS ARE HUMAN RIGHTS"
- board text added: "VA17"
- board text added: "~{CAS2}"
- board text added: "~{IPL0}"
- board text added: "~{IPL1}"
- board text added: "~{IPL2}"
- board text added: "~{LWR}"
- board text added: "~{NVRAM_RESET}"
- board text added: "~{UWR}"
- board text added: "~{VPA}"
- board text added: "®EPRO 2025"
- board text removed: "MADE BY COSAM"
- board text removed: "REPRO v1.2 BY COSAM"
- board text removed: "®EPRO 2023"
