File: MegaCD-837-8015-Rev0-MCE1/MegaCD.kicad_sch (KiCad schematic)
At the start: 126 parts, among them CN1 CON 25P ANGLE, CN2 EDGE 60P, CN3 CON 21P, IC1 68HC000, IC10 MB8464A-10L, IC11 TC511664BZ, IC12 TC511664BZ, IC13 65256BLFP-10T, IC14 65256BLFP-10T, IC15 LC8951, IC16 74HC00, IC17 MB8464A-90L, IC18 MB8464A-90L, IC19 74HC112, IC2 315-5477, IC20 74HC245, IC3 315-5476, IC4 27C1024, IC5 MB81C4256Z, IC5678 HM514270, IC6 MB81C4256Z, IC7 MB81C4256Z, IC8 MB81C4256Z, IC9 MB3790, J2 2TS, J3 MH, J4 CAS0, M0 TestPoint, M1 TestPoint, M10 TestPoint, M11 TestPoint, M2 TestPoint, M3 TestPoint, M4 TestPoint, M5 TestPoint, M6 TestPoint, M7 TestPoint, M8 TestPoint, M9 TestPoint

Commit message: Improve board design by making it possible to mostly manufacture at JLCPCB
Parts:
- C10, C11, C12, C13, C23, C28, C31, C37, C41, C42, C46, C9: footprint MegaCD_Footprints:CP_Elec_3x5.4 -> MegaCD_Footprints:CP_Elec_4x5.4
- C15, C16, C17, C18, C19, C20, C21, C22, C33, C35: now not fitted; now left out of the parts list
- C55: now not fitted
- IC16: footprint MegaCD_Footprints:SOIC-14W_5.3mm_P1.27mm -> MegaCD_Footprints:IC_SN74HC00DR
- IC19: footprint MegaCD_Footprints:SOIC-16W_5.3x10.2mm_P1.27mm -> MegaCD_Footprints:IC_SN74HC112DR
Connections:
- net OAD0: now reaches IC12.11 (D0), IC12.25 (A0), IC2.45 (OAD0)
- net OAD1: now reaches IC12.12 (D1), IC12.26 (A1), IC2.46 (OAD1)
- net OAD2: now reaches IC12.14 (D2), IC12.27 (A2), IC2.47 (OAD2)
- net OAD3: now reaches IC12.15 (D3), IC12.28 (A3), IC2.48 (OAD3)
- net OAD4: now reaches IC12.16 (D4), IC12.29 (A4), IC2.49 (OAD4)
- net OAD5: now reaches IC12.17 (D5), IC12.34 (A5), IC2.51 (OAD5)
- net OAD6: now reaches IC12.18 (D6), IC12.35 (A6), IC2.52 (OAD6)
- net OAD7: now reaches IC12.19 (D7), IC12.36 (A7), IC2.53 (OAD7)
- net OD8: now reaches IC12.2 (D8), IC2.54 (OD8)
- net OD9: now reaches IC12.3 (D9), IC2.55 (OD9)
- net OD10: now reaches IC12.4 (D10), IC2.56 (OD10)
- net OD11: now reaches IC12.5 (D11), IC2.57 (OD11)
- net OD12: now reaches IC12.6 (D12), IC2.58 (OD12)
- net OD13: now reaches IC12.7 (D13), IC2.59 (OD13)
- net OD14: now reaches IC12.8 (D14), IC2.62 (OD14)
- net OD15: now reaches IC12.9 (D15), IC2.63 (OD15)
- net LEDR: now reaches IC2.64 (LEDR), R6.1
- net LD1TRB: now reaches R6.2, TR2.1 (B)
- net ~{NVRAM_RESET}: now reaches IC10.26 (CS2), IC9.10 (~{RESET}), M0.1
- net NVRAM_VCC: now reaches C3.1, IC10.28 (VCC), IC9.3 (VOUT), IC9.4 (VOUT)
- net ~{RWE8951}: now reaches IC15.12 (~{RWE}), IC17.27 (~{WE}), IC18.27 (~{WE})
- net ~{ROE8951}: now reaches IC15.14 (~{ROE}), IC17.22 (~{OE}), IC18.22 (~{OE})
- net ~{RCS}: now reaches IC15.62 (~{RCS}), IC17.20 (~{CS1}), IC18.20 (~{CS1})
- net VCC2F: now reaches CN3.19 (Pin_19), CN3.2 (Pin_2), FB4.2
- net ~{RCS1Q}: now reaches IC16.2, IC19.5 (Q)
- net ~{RCS1N}: now reaches IC16.3, IC19.15 (~{R})
- net 25MF: now reaches FB5.1, IC2.1 (25M)
- net 12MF: now reaches FB1.2, IC2.129 (12M)
- net EAD0: now reaches IC11.11 (D0), IC11.25 (A0), IC2.17 (EAD0)
- net EAD1: now reaches IC11.12 (D1), IC11.26 (A1), IC2.18 (EAD1)
- net EAD2: now reaches IC11.14 (D2), IC11.27 (A2), IC2.19 (EAD2)
- net EAD3: now reaches IC11.15 (D3), IC11.28 (A3), IC2.20 (EAD3)
- net EAD4: now reaches IC11.16 (D4), IC11.29 (A4), IC2.21 (EAD4)
- net EAD5: now reaches IC11.17 (D5), IC11.34 (A5), IC2.22 (EAD5)
- net EAD6: now reaches IC11.18 (D6), IC11.35 (A6), IC2.23 (EAD6)
- net EAD7: now reaches IC11.19 (D7), IC11.36 (A7), IC2.24 (EAD7)
- net ED8: now reaches IC11.2 (D8), IC2.25 (ED8)
- net ED9: now reaches IC11.3 (D9), IC2.28 (ED9)
- net ED10: now reaches IC11.4 (D10), IC2.29 (ED10)
- net ED11: now reaches IC11.5 (D11), IC2.30 (ED11)
- net ED12: now reaches IC11.6 (D12), IC2.31 (ED12)
- net ED13: now reaches IC11.7 (D13), IC2.32 (ED13)
- net ED14: now reaches IC11.8 (D14), IC2.33 (ED14)
- net ED15: now reaches IC11.9 (D15), IC2.34 (ED15)
- net LEDG: now reaches IC2.65 (LEDG), R7.1
- net EXCK: now reaches CN1.17 (Pin_17), IC2.74 (EXCK)
- net C2PO: now reaches CN1.10 (Pin_10), IC2.77 (C2PO)
- net DB3: now reaches CN1.9 (Pin_9), IC2.78 (DB3)
- net DB2: now reaches CN1.8 (Pin_8), IC2.80 (DB2)
- net DB1: now reaches CN1.7 (Pin_7), IC2.81 (DB1)
- net DB0: now reaches CN1.6 (Pin_6), IC2.82 (DB0)
- net HDCK: now reaches CN1.5 (Pin_5), IC2.83 (HDCK)
- net ~{IRQ}: now reaches CN1.3 (Pin_3), IC2.86 (~{IRQ})
- net D/M: now reaches CN1.2 (Pin_2), IC2.87 (D/M)
- net ~{RWE}: now reaches IC13.27 (~{WE}), IC14.27 (~{WE}), IC3.63 (~{RWE})
- net LD1K: now reaches LD1.1 (K), TR2.3 (C)
- net LD1A: now reaches LD1.2 (A), R4.1
- net 50MF: now reaches FB2.1, OSC1.8 (OUT)
- net BATPW: now reaches C1.1, IC9.11 (CT)
- net LD2A: now reaches LD2.2 (A), R5.1
- net LD2TRB: now reaches R7.2, TR1.1 (B)
- net LD2K: now reaches LD2.1 (K), TR1.3 (C)
- net ~{RCS2N}: now reaches IC16.6, IC19.14 (~{R})
- net ~{RCS2Q}: now reaches IC16.5, IC19.9 (Q)
- net VBAT: now reaches BT1.1 (+), IC9.5 (VBAT2)
Other:
- moved on the sheet: CN1, FB2, FB5, R6, TR2
